Commit message: Rename baseplate

File: khi_duaro_description/urdf/duaro_macro_separation.xacro (robot description, xacro)
@@ -72,5 +72,5 @@
     </xacro:macro>
     <link name="${prefix}base_link"/>
-    <link name="${prefix}base_plate">
+    <link name="${prefix}khi_base_plate">
       <visual>
         <geometry>
@@ -112,5 +112,5 @@
       <origin xyz="0 0 0.0"/>
       <parent link="${prefix}base_link"/>
-      <child link="${prefix}base_plate"/>
+      <child link="${prefix}khi_base_plate"/>
     </joint>
     <!-- lower arm -->
